File: Voltage-sensor-mother-board.kicad_pcb (KiCad board)
At the start: 2 copper layers, 100 x 70 mm, 20 parts, among them J1 Conn_01x01_Female_M6_hole, J2 Conn_01x01_Female_M6_hole, J3 Conn_01x02_Male, J4 Conn_01x02_Female, J5 Conn_01x01_Female, J6 Conn_01x05_Female, J7 Conn_01x05_Female, M1 INA238_module, U1 CC1R5-xxxxSx-E, U2 AE-ADuM1250_module

Commit message: add v3.0
add v3.0
Parts:
- U2: moved to B.Cu
- turned U2 to 0 degrees
Connections:
- C1 pad 1: Net-(M1-Pad1) -> Net-(C1-Pad1)
- D1 pad 2: Net-(M1-Pad1) -> Net-(C1-Pad1)
- M1 pad 1: Net-(M1-Pad1) -> Net-(C1-Pad1)
- U1 pad 7: Net-(M1-Pad1) -> Net-(C1-Pad1)
- U2 pad 1: Net-(M1-Pad1) -> Net-(J6-Pad1)
- U2 pad 2: Net-(M1-Pad3) -> Net-(J6-Pad3)
- U2 pad 3: Net-(M1-Pad2) -> Net-(J6-Pad2)
- U2 pad 4: HVGND -> LVGND
- U2 pad 5: Net-(J6-Pad1) -> Net-(C1-Pad1)
- U2 pad 6: Net-(J6-Pad3) -> Net-(M1-Pad3)
- U2 pad 7: Net-(J6-Pad2) -> Net-(M1-Pad2)
- U2 pad 8: LVGND -> HVGND
Routing:
- net Net-(M1-Pad1): track 67.5 -> 0.00 mm, vias 3 -> 0
- net Net-(C1-Pad1): track 0.00 -> 67.5 mm, vias 0 -> 3
Other:
- board text added: "Voltage-sensor-mother 221130 V3.0"
- board text removed: "Voltage-sensor-mother 221025 V2.1"
Changed lines of the file:
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@@
   (title_block
     (title "Voltage sensor mother board")
-    (date "2022-10-25")
-    (rev "1.3")
+    (date "2022-11-30")
+    (rev "3.0")
     (company "teTra Aviaiton Corp.")
     (comment 1 "v1.2: fix AE-ADuM1250 size")
@@
     (comment 3 "v2.0: add LED and capacitor")
     (comment 4 "v2.1: fix edge cut 100.1 -> 100")
+    (comment 5 "v3.0: flip AE-Adum1250 module, side1 and side2")
   )
   (layers
@@
       (drillshape 0)
       (scaleselection 1)
-      (outputdirectory "Voltage-sensor-mother-board-v1p0/")
+      (outputdirectory "Voltage-sensor-mother-board-v3p0/")
     )
   )
@@
   (net 6 "Net-(J6-Pad2)")
   (net 7 "Net-(J6-Pad3)")
-  (net 8 "Net-(M1-Pad1)")
+  (net 8 "Net-(C1-Pad1)")
   (net 9 "Net-(M1-Pad2)")
   (net 10 "Net-(M1-Pad3)")
@@
     (pad "" thru_hole circle (at 3.175 7.62 180) (size 2 2) (drill 1) (layers *.Cu *.Mask))
     (pad "1" thru_hole oval (at 12.065 -5.08 180) (size 5 2) (drill 1 (offset 1 0)) (layers *.Cu *.Mask)
-      (net 8 "Net-(M1-Pad1)") (pinfunction "VSS") (pintype "input"))
+      (net 8 "Net-(C1-Pad1)") (pinfunction "VSS") (pintype "input"))
     (pad "2" thru_hole oval (at 12.065 -2.54 180) (size 5 2) (drill 1 (offset 1 0)) (layers *.Cu *.Mask)
       (net 9 "Net-(M1-Pad2)") (pinfunction "SCL") (pintype "input"))
@@
     )
   )
-  (footprint "kicad_teTra_footprint:AE-ADuM1250_module" (layer "F.Cu")
-    (at 81 99.62 180)
-    (property "Sheetfile" "Voltage-sensor-mother-board.kicad_sch")
-    (property "Sheetname" "")
-    (attr through_hole)
-    (fp_text reference "U2" (at -0.5 -18.5 180 unlocked) (layer "F.SilkS")
-      (effects (font (size 1 1) (thickness 0.15)))
-    )
-    (fp_text value "AE-ADuM1250_module" (at 0 18.5 180 unlocked) (layer "F.Fab")
-      (effects (font (size 1 1) (thickness 0.15)))
-    )
-    (fp_text user "${REFERENCE}" (at 0 20 180 unlocked) (layer "F.Fab")
-      (effects (font (size 1 1) (thickness 0.15)))
-    )
-    (fp_line (start -19 -9.5) (end -19 -17.5) (layer "F.SilkS") (width 0.12))
-    (fp_line (start 19 17.5) (end -19 17.5) (layer "F.SilkS") (width 0.12))
-    (fp_line (start 19 -17.5) (end 19 -9.5) (layer "F.SilkS") (width 0.12))
-    (fp_line (start -19 -17.5) (end 19 -17.5) (layer "F.SilkS") (width 0.12))
-    (fp_line (start 19 9.5) (end 19 17.5) (layer "F.SilkS") (width 0.12))
-    (fp_line (start -19 17.5) (end -19 9.5) (layer "F.SilkS") (width 0.12))
-    (fp_rect (start -18.5 -17) (end 18.5 17) (layer "Eco1.User") (width 0.12) (fill none))
-    (pad "" thru_hole circle (at 15.5 14 180) (size 6 6) (drill 3.2) (layers *.Cu *.Mask))
-    (pad "" thru_hole circle (at -15.5 -14 180) (size 6 6) (drill 3.2) (layers *.Cu *.Mask))
-    (pad "" thru_hole circle (at 15.5 -14 180) (size 6 6) (drill 3.2) (layers *.Cu *.Mask))
-    (pad "" thru_hole circle (at -15.5 14 180) (size 6 6) (drill 3.2) (layers *.Cu *.Mask))
-    (pad "1" thru_hole rect (at -14.5 -7.62 180) (size 10 3) (drill 1.5 (offset -3 0)) (layers *.Cu *.Mask)
-      (net 8 "Net-(M1-Pad1)") (pinfunction "VCC1") (pintype "input"))
-    (pad "2" thru_hole rect (at -14.5 -2.54 180) (size 10 3) (drill 1.5 (offset -3 0)) (layers *.Cu *.Mask)
-      (net 10 "Net-(M1-Pad3)") (pinfunction "SDA1") (pintype "bidirectional"))
-    (pad "3" thru_hole rect (at -14.5 2.54 180) (size 10 3) (drill 1.5 (offset -3 0)) (layers *.Cu *.Mask)
-      (net 9 "Net-(M1-Pad2)") (pinfunction "SCL1") (pintype "bidirectional"))
-    (pad "4" thru_hole rect (at -14.5 7.62 180) (size 10 3) (drill 1.5 (offset -3 0)) (layers *.Cu *.Mask)
-      (net 16 "HVGND") (pinfunction "GND1") (pintype "input"))
-    (pad "5" thru_hole rect (at 14.5 -7.62 180) (size 10 3) (drill 1.5 (offset 3 0)) (layers *.Cu *.Mask)
-      (net 5 "Net-(J6-Pad1)") (pinfunction "VCC2") (pintype "input"))
-    (pad "6" thru_hole rect (at 14.5 -2.54 180) (size 10 3) (drill 1.5 (offset 3 0)) (layers *.Cu *.Mask)
-      (net 7 "Net-(J6-Pad3)") (pinfunction "SDA2") (pintype "bidirectional"))
-    (pad "7" thru_hole rect (at 14.5 2.54 180) (size 10 3) (drill 1.5 (offset 3 0)) (layers *.Cu *.Mask)
-      (net 6 "Net-(J6-Pad2)") (pinfunction "SCL2") (pintype "bidirectional"))
-    (pad "8" thru_hole rect (at 14.5 7.62 180) (size 10 3) (drill 1.5 (offset 3 0)) (layers *.Cu *.Mask)
-      (net 15 "LVGND") (pinfunction "GND2") (pintype "input"))
-  )
   (footprint "kicad_teTra_footprint:CC1R5-4803SR-E" (layer "F.Cu")
     (at 123 100 180)
@@
       (net 14 "unconnected-(U1-Pad6)") (pinfunction "TRM") (pintype "input+no_connect"))
     (pad "7" smd roundrect (at 9.4 0 180) (size 3.2 1.2) (layers "F.Cu" "F.Paste" "F.Mask") (roundrect_rratio 0.25)
-      (net 8 "Net-(M1-Pad1)") (pinfunction "+Vout") (pintype "output"))
+      (net 8 "Net-(C1-Pad1)") (pinfunction "+Vout") (pintype "output"))
   )
   (footprint "LED_SMD:LED_0603_1608Metric_Pad1.05x0.95mm_HandSolder" (layer "F.Cu")
@@
       (net 17 "Net-(D1-Pad1)") (pinfunction "K") (pintype "passive"))
     (pad "2" smd roundrect locked (at 0.875 0 270) (size 1.05 0.95) (layers "F.Cu" "F.Paste" "F.Mask") (roundrect_rratio 0.25)
-      (net 8 "Net-(M1-Pad1)") (pinfunction "A") (pintype "passive"))
+      (net 8 "Net-(C1-Pad1)") (pinfunction "A") (pintype "passive"))
     (model "${KICAD6_3DMODEL_DIR}/LED_SMD.3dshapes/LED_0603_1608Metric.wrl"
       (offset (xyz 0 0 0))
@@
     (fp_line (start 0.8 0.4) (end -0.8 0.4) (layer "F.Fab") (width 0.1))
     (pad "1" smd roundrect locked (at -0.8625 0 90) (size 1.075 0.95) (layers "F.Cu" "F.Paste" "F.Mask") (roundrect_rratio 0.25)
-      (net 8 "Net-(M1-Pad1)") (pintype "passive"))
+      (net 8 "Net-(C1-Pad1)") (pintype "passive"))
     (pad "2" smd roundrect locked (at 0.8625 0 90) (size 1.075 0.95) (layers "F.Cu" "F.Paste" "F.Mask") (roundrect_rratio 0.25)
       (net 16 "HVGND") (pintype "passive"))
@@
     )
   )
+  (footprint "kicad_teTra_footprint:AE-ADuM1250_module" (layer "B.Cu")
+    (at 81 99.62)
+    (property "Sheetfile" "Voltage-sensor-mother-board.kicad_sch")
+    (property "Sheetname" "")
+    (attr through_hole)
+    (fp_text reference "U2" (at -0.5 18.5 180 unlocked) (layer "B.SilkS")
+      (effects (font (size 1 1) (thickness 0.15)) (justify mirror))
+    )
+    (fp_text value "AE-ADuM1250_module" (at 0 -18.5 180 unlocked) (layer "B.Fab")
+      (effects (font (size 1 1) (thickness 0.15)) (justify mirror))
+    )
+    (fp_text user "${REFERENCE}" (at 0 -20 180 unlocked) (layer "B.Fab")
+      (effects (font (size 1 1) (thickness 0.15)) (justify mirror))
+    )
+    (fp_line (start -19 9.5) (end -19 17.5) (layer "B.SilkS") (width 0.12))
+    (fp_line (start 19 -17.5) (end -19 -17.5) (layer "B.SilkS") (width 0.12))
+    (fp_line (start 19 17.5) (end 19 9.5) (layer "B.SilkS") (width 0.12))
+    (fp_line (start -19 17.5) (end 19 17.5) (layer "B.SilkS") (width 0.12))
+    (fp_line (start 19 -9.5) (end 19 -17.5) (layer "B.SilkS") (width 0.12))
+    (fp_line (start -19 -17.5) (end -19 -9.5) (layer "B.SilkS") (width 0.12))
+    (fp_rect (start -18.5 17) (end 18.5 -17) (layer "Eco1.User") (width 0.12) (fill none))
+    (pad "" thru_hole circle (at 15.5 -14) (size 6 6) (drill 3.2) (layers *.Cu *.Mask))
+    (pad "" thru_hole circle (at -15.5 14) (size 6 6) (drill 3.2) (layers *.Cu *.Mask))
+    (pad "" thru_hole circle (at 15.5 14) (size 6 6) (drill 3.2) (layers *.Cu *.Mask))
+    (pad "" thru_hole circle (at -15.5 -14) (size 6 6) (drill 3.2) (layers *.Cu *.Mask))
+    (pad "1" thru_hole rect (at -14.5 7.62) (size 10 3) (drill 1.5 (offset -3 0)) (layers *.Cu *.Mask)
+      (net 5 "Net-(J6-Pad1)") (pinfunction "VCC1") (pintype "input"))
+    (pad "2" thru_hole rect (at -14.5 2.54) (size 10 3) (drill 1.5 (offset -3 0)) (layers *.Cu *.Mask)
+      (net 7 "Net-(J6-Pad3)") (pinfunction "SDA1") (pintype "bidirectional"))
+    (pad "3" thru_hole rect (at -14.5 -2.54) (size 10 3) (drill 1.5 (offset -3 0)) (layers *.Cu *.Mask)
+      (net 6 "Net-(J6-Pad2)") (pinfunction "SCL1") (pintype "bidirectional"))
+    (pad "4" thru_hole rect (at -14.5 -7.62) (size 10 3) (drill 1.5 (offset -3 0)) (layers *.Cu *.Mask)
+      (net 15 "LVGND") (pinfunction "GND1") (pintype "input"))
+    (pad "5" thru_hole rect (at 14.5 7.62) (size 10 3) (drill 1.5 (offset 3 0)) (layers *.Cu *.Mask)
+      (net 8 "Net-(C1-Pad1)") (pinfunction "VCC2") (pintype "input"))
+    (pad "6" thru_hole rect (at 14.5 2.54) (size 10 3) (drill 1.5 (offset 3 0)) (layers *.Cu *.Mask)
+      (net 10 "Net-(M1-Pad3)") (pinfunction "SDA2") (pintype "bidirectional"))
+    (pad "7" thru_hole rect (at 14.5 -2.54) (size 10 3) (drill 1.5 (offset 3 0)) (layers *.Cu *.Mask)
+      (net 9 "Net-(M1-Pad2)") (pinfunction "SCL2") (pintype "bidirectional"))
+    (pad "8" thru_hole rect (at 14.5 -7.62) (size 10 3) (drill 1.5 (offset 3 0)) (layers *.Cu *.Mask)
+      (net 16 "HVGND") (pinfunction "GND2") (pintype "input"))
+  )
   (gr_rect (start 150 65) (end 136 120) (layer "Eco1.User") (width 0.15) (fill none))
   (gr_rect (start 150 120) (end 50 50) (layer "Eco1.User") (width 0.15) (fill none))
@@
     (effects (font (size 1 1) (thickness 0.15)))
   )
-  (gr_text "Voltage-sensor-mother\n221025 V2.1" (at 53 67) (layer "F.SilkS")
+  (gr_text "Voltage-sensor-mother\n221130 V3.0" (at 53 67) (layer "F.SilkS")
     (effects (font (size 1 1) (thickness 0.15)) (justify left))
   )
