File: Voltage-sensor-mother-board.kicad_sch (KiCad schematic)
At the start: 20 parts, among them J1 Conn_01x01_Female_M6_hole, J2 Conn_01x01_Female_M6_hole, J3 Conn_01x02_Male, J4 Conn_01x02_Female, J5 Conn_01x01_Female, J6 Conn_01x05_Female, J7 Conn_01x05_Female, M1 INA238_module, U1 CC1R5-xxxxSx-E, U2 AE-ADuM1250_module

Commit message: add v3.0
add v3.0
Connections:
- net HVGND: now also U2.8 (GND2); no longer U2.4 (GND1)
- net LVGND: now also U2.4 (GND1); no longer U2.8 (GND2)
- net at C1.1, D1.2 (A), M1.1 (VSS)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: now also U2.5 (VCC2); no longer U2.1 (VCC1)
- net at U2.2 (SDA1): now also J6.3 (Pin_3), J7.2 (Pin_2); no longer M1.3 (SDA)
- net at U2.3 (SCL1): now also J6.2 (Pin_2), J7.3 (Pin_3); no longer M1.2 (SCL)
- net at J6.1 (Pin_1), J7.1 (Pin_1): now also U2.1 (VCC1); no longer U2.5 (VCC2)
- new net: M1.3 (SDA), U2.6 (SDA2)
- new net: M1.2 (SCL), U2.7 (SCL2)
Changed lines of the file:
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@@
   (title_block
     (title "Voltage sensor mother board")
-    (date "2022-10-25")
-    (rev "2.0")
+    (date "2022-11-30")
+    (rev "3.0")
     (company "teTra Aviation Corp.")
     (comment 1 "v2.0: add LED and Capacitor")
+    (comment 2 "v3.0: flip AE-Adum1250 module, side1 and side2")
   )
   (junction (at 122.555 115.57) (diameter 0) (color 0 0 0 0)
@@
     )
   )
-  (symbol (lib_id "kicad6_teTra_library:AE-ADuM1250_module") (at 200.025 76.835 0) (unit 1)
+  (symbol (lib_id "kicad6_teTra_library:AE-ADuM1250_module") (at 199.39 76.835 0) (mirror y) (unit 1)
     (in_bom yes) (on_board yes) (fields_autoplaced)
     (property "Reference" "U2" (id 0) (at 199.7075 66.04 0))
     (property "Value" "AE-ADuM1250_module" (id 1) (at 199.7075 68.58 0))
-    (property "Footprint" "kicad_teTra_footprint:AE-ADuM1250_module" (id 2) (at 200.025 70.485 0)
-      (effects (font (size 1.27 1.27)) hide)
-    )
-    (property "Datasheet" "" (id 3) (at 200.025 70.485 0)
-      (effects (font (size 1.27 1.27)) hide)
-    )
+    (property "Footprint" "kicad_teTra_footprint:AE-ADuM1250_module" (id 2) (at 199.39 70.485 0)
+      (effects (font (size 1.27 1.27)) hide)
+    )
+    (property "Datasheet" "" (id 3) (at 199.39 70.485 0)
+      (effects (font (size 1.27 1.27)) hide)
+    )
